Commit message: Realsense camera added

File: mir_robot/mir_description/urdf/include/mir_250_v1.urdf.xacro (robot description, xacro)
@@ -6,5 +6,5 @@
   <xacro:include filename="$(find mir_description)/urdf/include/wheel.urdf.xacro" />
   <xacro:include filename="$(find mir_description)/urdf/include/caster.urdf.xacro" />
-  <xacro:include filename="$(find realsense2_description)/urdf/_d435i.urdf.xacro"/>
+  <!-- <xacro:include filename="$(find realsense2_description)/urdf/_d435i.urdf.xacro"/> -->
   <xacro:include filename="$(find robotiq_description)/urdf/robotiq_85_gripper.urdf.xacro"/>
   <xacro:property name="deg_to_rad" value="0.017453293" />
@@ -314,7 +314,12 @@
       <origin xyz="0.035 0.05 0.03" rpy="0 ${pi} ${0.5 * pi}" />
     </joint>
-    <xacro:sensor_d435i parent="ur_flange" name="realsense" use_nominal_extrinsics="true">
+    <!-- <xacro:sensor_d435i parent="ur_flange" name="realsense" use_nominal_extrinsics="true">
       <origin xyz="0.02 0 -0.061" rpy="${pi} 0 0"/>
-    </xacro:sensor_d435i>
+    </xacro:sensor_d435i> -->
+    <xacro:include filename="$(find realsense_ros2_gazebo)/xacro/depthcam.xacro"/>
+    <xacro:realsense_d435 sensor_name="d435" parent_link="ur_flange" rate="10">
+      <origin rpy="${pi} 0 0" xyz="0.02 0 -0.061"/>
+      <!-- <origin rpy="0 0 0 " xyz="0 0 0"/> -->
+    </xacro:realsense_d435>
     <!-- <link name="robotiq_coupler">
       <visual>

File: realsense2_description/urdf/_d435.urdf.xacro (robot description, xacro)
@@ -150,4 +150,131 @@
       </xacro:usb_plug>
     </xacro:if>
+    <!-- gazebo plugin -->
+    <xacro:property name="deg_to_rad" value="0.01745329251994329577" />
+    <xacro:property name="sensor_name" value="d435" />
+    <xacro:property name="rate" value="10" />
+    <gazebo reference="${sensor_name}_link">
+      <self_collide>0</self_collide>
+      <enable_wind>0</enable_wind>
+      <kinematic>0</kinematic>
+      <gravity>1</gravity>
+      <mu2>1</mu2>
+      <fdir1>0 0 0</fdir1>
+      <kp>1e+13</kp>
+      <kd>1</kd>
+      <sensor name="${sensor_name}_color" type="camera">
+        <camera name="${sensor_name}">
+          <horizontal_fov>${69.4*deg_to_rad}</horizontal_fov>
+          <image>
+            <width>640</width>
+            <height>480</height>
+            <format>RGB_INT8</format>
+          </image>
+          <clip>
+            <near>0.1</near>
+            <far>100</far>
+          </clip>
+          <noise>
+            <type>gaussian</type>
+            <mean>0.0</mean>
+            <stddev>0.007</stddev>
+          </noise>
+        </camera>
+        <always_on>1</always_on>
+        <update_rate>30</update_rate>
+        <visualize>1</visualize>
+      </sensor>
+      <sensor name="${sensor_name}_ired1" type="camera">
+        <camera name="${sensor_name}">
+          <horizontal_fov>${85.2*deg_to_rad}</horizontal_fov>
+          <image>
+            <width>1280</width>
+            <height>720</height>
+            <format>L_INT8</format>
+          </image>
+          <clip>
+            <near>0.1</near>
+            <far>100</far>
+          </clip>
+          <noise>
+            <type>gaussian</type>
+            <mean>0.0</mean>
+            <stddev>0.05</stddev>
+          </noise>
+        </camera>
+        <always_on>1</always_on>
+        <update_rate>90</update_rate>
+        <visualize>0</visualize>
+      </sensor>
+      <sensor name="${sensor_name}_ired2" type="camera">
+        <camera name="${sensor_name}">
+          <horizontal_fov>${85.2*deg_to_rad}</horizontal_fov>
+          <image>
+            <width>1280</width>
+            <height>720</height>
+            <format>L_INT8</format>
+          </image>
+          <clip>
+            <near>0.1</near>
+            <far>100</far>
+          </clip>
+          <noise>
+            <type>gaussian</type>
+            <mean>0.0</mean>
+            <stddev>0.05</stddev>
+          </noise>
+        </camera>
+        <always_on>1</always_on>
+        <update_rate>90</update_rate>
+        <visualize>0</visualize>
+      </sensor>
+      <sensor name="${sensor_name}_depth" type="depth">
+        <camera name="${sensor_name}">
+          <horizontal_fov>${85.2*deg_to_rad}</horizontal_fov>
+          <image>
+            <width>1280</width>
+            <height>720</height>
+          </image>
+          <clip>
+            <near>0.1</near>
+            <far>100</far>
+          </clip>
+          <noise>
+            <type>gaussian</type>
+            <mean>0.0</mean>
+            <stddev>0.100</stddev>
+          </noise>
+        </camera>
+        <always_on>1</always_on>
+        <update_rate>90</update_rate>
+        <visualize>0</visualize>
+      </sensor>
+    </gazebo>
+    <gazebo>
+      <plugin name="${sensor_name}" filename="librealsense_gazebo_plugin.so">
+        <prefix>${sensor_name}_</prefix>
+        <depthUpdateRate>${rate}</depthUpdateRate>
+        <colorUpdateRate>${rate}</colorUpdateRate>
+        <infraredUpdateRate>${rate}</infraredUpdateRate>
+        <depthTopicName>depth/image_raw</depthTopicName>
+        <depthCameraInfoTopicName>depth/camera_info</depthCameraInfoTopicName>
+        <colorTopicName>color/image_raw</colorTopicName>
+        <colorCameraInfoTopicName>color/camera_info</colorCameraInfoTopicName>
+        <infrared1TopicName>infra1/image_raw</infrared1TopicName>
+        <infrared1CameraInfoTopicName>infra1/camera_info</infrared1CameraInfoTopicName>
+        <infrared2TopicName>infra2/image_raw</infrared2TopicName>
+        <infrared2CameraInfoTopicName>infra2/camera_info</infrared2CameraInfoTopicName>
+        <colorOpticalframeName>${sensor_name}_color_optical_frame</colorOpticalframeName>
+        <depthOpticalframeName>${sensor_name}_depth_optical_frame</depthOpticalframeName>
+        <infrared1OpticalframeName>${sensor_name}_infrared1_optical_frame</infrared1OpticalframeName>
+        <infrared2OpticalframeName>${sensor_name}_infrared2_optical_frame</infrared2OpticalframeName>
+        <rangeMinDepth>0.2</rangeMinDepth>
+        <rangeMaxDepth>10.0</rangeMaxDepth>
+        <pointCloud>false</pointCloud>
+        <pointCloudTopicName>depth/color/points</pointCloudTopicName>
+        <pointCloudCutoff>0.25</pointCloudCutoff>
+        <pointCloudCutoffMax>9.0</pointCloudCutoffMax>
+      </plugin>
+    </gazebo>
   </xacro:macro>
 </robot>

Commit message: Realsense plugin working with description file and interactive marker issue resolved temp

File: mir_robot/mir_description/urdf/include/mir_250_v1.urdf.xacro (robot description, xacro)
@@ -6,5 +6,5 @@
   <xacro:include filename="$(find mir_description)/urdf/include/wheel.urdf.xacro" />
   <xacro:include filename="$(find mir_description)/urdf/include/caster.urdf.xacro" />
-  <!-- <xacro:include filename="$(find realsense2_description)/urdf/_d435i.urdf.xacro"/> -->
+  <xacro:include filename="$(find realsense2_description)/urdf/_d435i.urdf.xacro"/>
   <xacro:include filename="$(find robotiq_description)/urdf/robotiq_85_gripper.urdf.xacro"/>
   <xacro:property name="deg_to_rad" value="0.017453293" />
@@ -222,11 +222,10 @@
     <xacro:property name="initial_positions_file" default="$(arg initial_positions_file)"/>
     <!-- create link fixed to the "world" -->
-    <!-- <link name="world" />
+    <link name="world" />
     <joint name="world_joint" type="fixed">
       <parent link="${prefix}base_link" />
       <child link="world" />
       <origin xyz="0.135 0 0.79" rpy="0 0 ${0.5 * pi}" />
-    </joint> -->
-    <!-- ${prefix}base_link -->
+    </joint>
     <!-- arm -->
     <xacro:ur_robot
@@ -271,6 +270,6 @@
     <xacro:if value="$(arg sim_gazebo)">
       <!-- Gazebo plugins -->
-      <!-- <gazebo reference="world">
-      </gazebo> -->
+      <gazebo reference="world">
+      </gazebo>
       <gazebo>
         <plugin filename="libgazebo_ros2_control.so" name="gazebo_ros2_control_ur">
@@ -285,6 +284,6 @@
     <xacro:if value="$(arg sim_ignition)">
       <!-- Gazebo plugins -->
-      <!-- <gazebo reference="world">
-      </gazebo> -->
+      <gazebo reference="world">
+      </gazebo>
       <gazebo>
         <plugin filename="libign_ros2_control-system.so" name="ign_ros2_control::IgnitionROS2ControlPlugin">
@@ -314,12 +313,7 @@
       <origin xyz="0.035 0.05 0.03" rpy="0 ${pi} ${0.5 * pi}" />
     </joint>
-    <!-- <xacro:sensor_d435i parent="ur_flange" name="realsense" use_nominal_extrinsics="true">
+    <xacro:sensor_d435i parent="ur_flange" name="realsense" use_nominal_extrinsics="true">
       <origin xyz="0.02 0 -0.061" rpy="${pi} 0 0"/>
-    </xacro:sensor_d435i> -->
-    <xacro:include filename="$(find realsense_ros2_gazebo)/xacro/depthcam.xacro"/>
-    <xacro:realsense_d435 sensor_name="d435" parent_link="ur_flange" rate="10">
-      <origin rpy="${pi} 0 0" xyz="0.02 0 -0.061"/>
-      <!-- <origin rpy="0 0 0 " xyz="0 0 0"/> -->
-    </xacro:realsense_d435>
+    </xacro:sensor_d435i>
     <!-- <link name="robotiq_coupler">
       <visual>

File: realsense2_description/urdf/_d435.urdf.xacro (robot description, xacro)
@@ -150,131 +150,4 @@
       </xacro:usb_plug>
     </xacro:if>
-    <!-- gazebo plugin -->
-    <xacro:property name="deg_to_rad" value="0.01745329251994329577" />
-    <xacro:property name="sensor_name" value="d435" />
-    <xacro:property name="rate" value="10" />
-    <gazebo reference="${sensor_name}_link">
-      <self_collide>0</self_collide>
-      <enable_wind>0</enable_wind>
-      <kinematic>0</kinematic>
-      <gravity>1</gravity>
-      <mu2>1</mu2>
-      <fdir1>0 0 0</fdir1>
-      <kp>1e+13</kp>
-      <kd>1</kd>
-      <sensor name="${sensor_name}_color" type="camera">
-        <camera name="${sensor_name}">
-          <horizontal_fov>${69.4*deg_to_rad}</horizontal_fov>
-          <image>
-            <width>640</width>
-            <height>480</height>
-            <format>RGB_INT8</format>
-          </image>
-          <clip>
-            <near>0.1</near>
-            <far>100</far>
-          </clip>
-          <noise>
-            <type>gaussian</type>
-            <mean>0.0</mean>
-            <stddev>0.007</stddev>
-          </noise>
-        </camera>
-        <always_on>1</always_on>
-        <update_rate>30</update_rate>
-        <visualize>1</visualize>
-      </sensor>
-      <sensor name="${sensor_name}_ired1" type="camera">
-        <camera name="${sensor_name}">
-          <horizontal_fov>${85.2*deg_to_rad}</horizontal_fov>
-          <image>
-            <width>1280</width>
-            <height>720</height>
-            <format>L_INT8</format>
-          </image>
-          <clip>
-            <near>0.1</near>
-            <far>100</far>
-          </clip>
-          <noise>
-            <type>gaussian</type>
-            <mean>0.0</mean>
-            <stddev>0.05</stddev>
-          </noise>
-        </camera>
-        <always_on>1</always_on>
-        <update_rate>90</update_rate>
-        <visualize>0</visualize>
-      </sensor>
-      <sensor name="${sensor_name}_ired2" type="camera">
-        <camera name="${sensor_name}">
-          <horizontal_fov>${85.2*deg_to_rad}</horizontal_fov>
-          <image>
-            <width>1280</width>
-            <height>720</height>
-            <format>L_INT8</format>
-          </image>
-          <clip>
-            <near>0.1</near>
-            <far>100</far>
-          </clip>
-          <noise>
-            <type>gaussian</type>
-            <mean>0.0</mean>
-            <stddev>0.05</stddev>
-          </noise>
-        </camera>
-        <always_on>1</always_on>
-        <update_rate>90</update_rate>
-        <visualize>0</visualize>
-      </sensor>
-      <sensor name="${sensor_name}_depth" type="depth">
-        <camera name="${sensor_name}">
-          <horizontal_fov>${85.2*deg_to_rad}</horizontal_fov>
-          <image>
-            <width>1280</width>
-            <height>720</height>
-          </image>
-          <clip>
-            <near>0.1</near>
-            <far>100</far>
-          </clip>
-          <noise>
-            <type>gaussian</type>
-            <mean>0.0</mean>
-            <stddev>0.100</stddev>
-          </noise>
-        </camera>
-        <always_on>1</always_on>
-        <update_rate>90</update_rate>
-        <visualize>0</visualize>
-      </sensor>
-    </gazebo>
-    <gazebo>
-      <plugin name="${sensor_name}" filename="librealsense_gazebo_plugin.so">
-        <prefix>${sensor_name}_</prefix>
-        <depthUpdateRate>${rate}</depthUpdateRate>
-        <colorUpdateRate>${rate}</colorUpdateRate>
-        <infraredUpdateRate>${rate}</infraredUpdateRate>
-        <depthTopicName>depth/image_raw</depthTopicName>
-        <depthCameraInfoTopicName>depth/camera_info</depthCameraInfoTopicName>
-        <colorTopicName>color/image_raw</colorTopicName>
-        <colorCameraInfoTopicName>color/camera_info</colorCameraInfoTopicName>
-        <infrared1TopicName>infra1/image_raw</infrared1TopicName>
-        <infrared1CameraInfoTopicName>infra1/camera_info</infrared1CameraInfoTopicName>
-        <infrared2TopicName>infra2/image_raw</infrared2TopicName>
-        <infrared2CameraInfoTopicName>infra2/camera_info</infrared2CameraInfoTopicName>
-        <colorOpticalframeName>${sensor_name}_color_optical_frame</colorOpticalframeName>
-        <depthOpticalframeName>${sensor_name}_depth_optical_frame</depthOpticalframeName>
-        <infrared1OpticalframeName>${sensor_name}_infrared1_optical_frame</infrared1OpticalframeName>
-        <infrared2OpticalframeName>${sensor_name}_infrared2_optical_frame</infrared2OpticalframeName>
-        <rangeMinDepth>0.2</rangeMinDepth>
-        <rangeMaxDepth>10.0</rangeMaxDepth>
-        <pointCloud>false</pointCloud>
-        <pointCloudTopicName>depth/color/points</pointCloudTopicName>
-        <pointCloudCutoff>0.25</pointCloudCutoff>
-        <pointCloudCutoffMax>9.0</pointCloudCutoffMax>
-      </plugin>
-    </gazebo>
   </xacro:macro>
 </robot>

File: realsense2_description/urdf/_d435i.urdf.xacro (robot description, xacro)
@@ -22,4 +22,5 @@
   <xacro:include filename="$(find realsense2_description)/urdf/_d435.urdf.xacro"/>
   <xacro:include filename="$(find realsense2_description)/urdf/_d435i_imu_modules.urdf.xacro"/>
+  <xacro:include filename="$(find realsense2_description)/urdf/_d435i_gazebo.xacro"/>
   <xacro:macro name="sensor_d435i" params="parent *origin name:=camera use_nominal_extrinsics:=false">
     <xacro:sensor_d435 parent="${parent}" name="${name}" use_nominal_extrinsics="${use_nominal_extrinsics}">
@@ -27,4 +28,30 @@
     </xacro:sensor_d435>
     <xacro:d435i_imu_modules name="${name}" use_nominal_extrinsics="${use_nominal_extrinsics}"/>
+    <xacro:gazebo_d435i camera_name="${name}"
+                        topics_ns="camera"
+                        reference_link="${name}_link"
+                        depth_optical_frame="${name}_depth_optical_frame"
+                        depth_width="848"
+                        depth_height="480"
+                        depth_fps="60"
+                        color_optical_frame="${name}_color_optical_frame"
+                        color_width="1920"
+                        color_height="1080"
+                        color_fps="30"
+                        infrared1_optical_frame="${name}_left_ir_optical_frame"
+                        infrared2_optical_frame="${name}_right_ir_optical_frame"
+                        infra_width="848"
+                        infra_height="480"
+                        infra_fps="60"
+                        accel_optical_frame="${name}_accel_optical_frame"
+                        gyro_optical_frame="${name}_gyro_optical_frame"
+                        accel_fps="63"
+                        gyro_fps="200"
+                        enable_pointCloud="true"
+                        unite_imu_method="linear_interpolation"
+                        clip_distance="-1.0"
+                        align_depth="false"
+                        visualize="true"
+    />
   </xacro:macro>
 </robot>

File: realsense2_description/urdf/_d435i_gazebo.xacro (robot description, xacro)
@@ -1,12 +1,21 @@
+<?xml version="1.0"?>
+<!--
+Aknolegment: This file was originally copied from the realsense repository of
+pal-robotics-forks( https://github.com/pal-robotics-forks/realsense/ )
+and then modified.
+License: Apache 2.0. See LICENSE file in root directory.
+Copyright(c) 2017 PAL Robotics, S.L. All Rights Reserved
+This is the Gazebo URDF model for the Intel RealSense D435i camera
+-->
 <robot xmlns:xacro="http://ros.org/wiki/xacro">
     <xacro:macro name="gazebo_d435i" params=" reference_link
                                             camera_name:=camera
                                             topics_ns:=camera
-                                            depth_optical_frame
-                                            color_optical_frame
-                                            infrared1_optical_frame
-                                            infrared2_optical_frame
-                                            accel_optical_frame
-                                            gyro_optical_frame
+                                            depth_optical_frame:=camera_depth_optical_frame
+                                            color_optical_frame:=camera_color_optical_frame
+                                            infrared1_optical_frame:=camera__left_ir_optical_frame
+                                            infrared2_optical_frame:=camera__right_ir_optical_frame
+                                            accel_optical_frame:=camera_accel_optical_frame
+                                            gyro_optical_frame:=camera_gyro_optical_frame
                                             visualize:=false
                                             align_depth:=false
