Commit message: Aruco to Nav2 goal

File: Universal_Robots_ROS2_Description/urdf/inc/ur_common.xacro (robot description, xacro)
@@ -52,28 +52,28 @@
     <xacro:property name="sec_kinematics" value="${config_kinematics_parameters['kinematics']}" />
     <!-- JOINTS LIMIT PARAMETERS -->
-    <xacro:property name="shoulder_pan_lower_limit" value="${sec_limits['shoulder_pan_joint']['min_position']}" scope="parent"/>
-    <xacro:property name="shoulder_pan_upper_limit" value="${sec_limits['shoulder_pan_joint']['max_position']}" scope="parent"/>
-    <xacro:property name="shoulder_pan_velocity_limit" value="${sec_limits['shoulder_pan_joint']['max_velocity']}" scope="parent"/>
-    <xacro:property name="shoulder_pan_effort_limit" value="${sec_limits['shoulder_pan_joint']['max_effort']}" scope="parent"/>
-    <xacro:property name="shoulder_lift_lower_limit" value="${sec_limits['shoulder_lift_joint']['min_position']}" scope="parent"/>
-    <xacro:property name="shoulder_lift_upper_limit" value="${sec_limits['shoulder_lift_joint']['max_position']}" scope="parent"/>
-    <xacro:property name="shoulder_lift_velocity_limit" value="${sec_limits['shoulder_lift_joint']['max_velocity']}" scope="parent"/>
-    <xacro:property name="shoulder_lift_effort_limit" value="${sec_limits['shoulder_lift_joint']['max_effort']}" scope="parent"/>
-    <xacro:property name="elbow_joint_lower_limit" value="${sec_limits['elbow_joint']['min_position']}" scope="parent"/>
-    <xacro:property name="elbow_joint_upper_limit" value="${sec_limits['elbow_joint']['max_position']}" scope="parent"/>
-    <xacro:property name="elbow_joint_velocity_limit" value="${sec_limits['elbow_joint']['max_velocity']}" scope="parent"/>
-    <xacro:property name="elbow_joint_effort_limit" value="${sec_limits['elbow_joint']['max_effort']}" scope="parent"/>
-    <xacro:property name="wrist_1_lower_limit" value="${sec_limits['wrist_1_joint']['min_position']}" scope="parent"/>
-    <xacro:property name="wrist_1_upper_limit" value="${sec_limits['wrist_1_joint']['max_position']}" scope="parent"/>
-    <xacro:property name="wrist_1_velocity_limit" value="${sec_limits['wrist_1_joint']['max_velocity']}" scope="parent"/>
-    <xacro:property name="wrist_1_effort_limit" value="${sec_limits['wrist_1_joint']['max_effort']}" scope="parent"/>
-    <xacro:property name="wrist_2_lower_limit" value="${sec_limits['wrist_2_joint']['min_position']}" scope="parent"/>
-    <xacro:property name="wrist_2_upper_limit" value="${sec_limits['wrist_2_joint']['max_position']}" scope="parent"/>
-    <xacro:property name="wrist_2_velocity_limit" value="${sec_limits['wrist_2_joint']['max_velocity']}" scope="parent"/>
-    <xacro:property name="wrist_2_effort_limit" value="${sec_limits['wrist_2_joint']['max_effort']}" scope="parent"/>
-    <xacro:property name="wrist_3_lower_limit" value="${sec_limits['wrist_3_joint']['min_position']}" scope="parent"/>
-    <xacro:property name="wrist_3_upper_limit" value="${sec_limits['wrist_3_joint']['max_position']}" scope="parent"/>
-    <xacro:property name="wrist_3_velocity_limit" value="${sec_limits['wrist_3_joint']['max_velocity']}" scope="parent"/>
-    <xacro:property name="wrist_3_effort_limit" value="${sec_limits['wrist_3_joint']['max_effort']}" scope="parent"/>
+    <xacro:property name="shoulder_pan_lower_limit" value="${sec_limits['ur_shoulder_pan_joint']['min_position']}" scope="parent"/>
+    <xacro:property name="shoulder_pan_upper_limit" value="${sec_limits['ur_shoulder_pan_joint']['max_position']}" scope="parent"/>
+    <xacro:property name="shoulder_pan_velocity_limit" value="${sec_limits['ur_shoulder_pan_joint']['max_velocity']}" scope="parent"/>
+    <xacro:property name="shoulder_pan_effort_limit" value="${sec_limits['ur_shoulder_pan_joint']['max_effort']}" scope="parent"/>
+    <xacro:property name="shoulder_lift_lower_limit" value="${sec_limits['ur_shoulder_lift_joint']['min_position']}" scope="parent"/>
+    <xacro:property name="shoulder_lift_upper_limit" value="${sec_limits['ur_shoulder_lift_joint']['max_position']}" scope="parent"/>
+    <xacro:property name="shoulder_lift_velocity_limit" value="${sec_limits['ur_shoulder_lift_joint']['max_velocity']}" scope="parent"/>
+    <xacro:property name="shoulder_lift_effort_limit" value="${sec_limits['ur_shoulder_lift_joint']['max_effort']}" scope="parent"/>
+    <xacro:property name="elbow_joint_lower_limit" value="${sec_limits['ur_elbow_joint']['min_position']}" scope="parent"/>
+    <xacro:property name="elbow_joint_upper_limit" value="${sec_limits['ur_elbow_joint']['max_position']}" scope="parent"/>
+    <xacro:property name="elbow_joint_velocity_limit" value="${sec_limits['ur_elbow_joint']['max_velocity']}" scope="parent"/>
+    <xacro:property name="elbow_joint_effort_limit" value="${sec_limits['ur_elbow_joint']['max_effort']}" scope="parent"/>
+    <xacro:property name="wrist_1_lower_limit" value="${sec_limits['ur_wrist_1_joint']['min_position']}" scope="parent"/>
+    <xacro:property name="wrist_1_upper_limit" value="${sec_limits['ur_wrist_1_joint']['max_position']}" scope="parent"/>
+    <xacro:property name="wrist_1_velocity_limit" value="${sec_limits['ur_wrist_1_joint']['max_velocity']}" scope="parent"/>
+    <xacro:property name="wrist_1_effort_limit" value="${sec_limits['ur_wrist_1_joint']['max_effort']}" scope="parent"/>
+    <xacro:property name="wrist_2_lower_limit" value="${sec_limits['ur_wrist_2_joint']['min_position']}" scope="parent"/>
+    <xacro:property name="wrist_2_upper_limit" value="${sec_limits['ur_wrist_2_joint']['max_position']}" scope="parent"/>
+    <xacro:property name="wrist_2_velocity_limit" value="${sec_limits['ur_wrist_2_joint']['max_velocity']}" scope="parent"/>
+    <xacro:property name="wrist_2_effort_limit" value="${sec_limits['ur_wrist_2_joint']['max_effort']}" scope="parent"/>
+    <xacro:property name="wrist_3_lower_limit" value="${sec_limits['ur_wrist_3_joint']['min_position']}" scope="parent"/>
+    <xacro:property name="wrist_3_upper_limit" value="${sec_limits['ur_wrist_3_joint']['max_position']}" scope="parent"/>
+    <xacro:property name="wrist_3_velocity_limit" value="${sec_limits['ur_wrist_3_joint']['max_velocity']}" scope="parent"/>
+    <xacro:property name="wrist_3_effort_limit" value="${sec_limits['ur_wrist_3_joint']['max_effort']}" scope="parent"/>
     <!-- DH PARAMETERS -->
     <xacro:property name="d1" value="${sec_dh_parameters['d1']}" scope="parent"/>

File: Universal_Robots_ROS2_Description/urdf/ur.ros2_control.xacro (robot description, xacro)
@@ -7,5 +7,5 @@
     sim_ignition:=false
     headless_mode:=false
-    initial_positions:=${dict(shoulder_pan_joint=0.0,shoulder_lift_joint=-1.57,elbow_joint=0.0,wrist_1_joint=-1.57,wrist_2_joint=0.0,wrist_3_joint=0.0)}
+    initial_positions:=${dict(ur_shoulder_pan_joint=0.0,ur_shoulder_lift_joint=-1.57,ur_elbow_joint=0.0,ur_wrist_1_joint=-1.57,ur_wrist_2_joint=0.0,ur_wrist_3_joint=0.0)}
     use_tool_communication:=false
     script_filename output_recipe_filename
@@ -75,5 +75,5 @@
         <state_interface name="position">
           <!-- initial position for the FakeSystem and simulation -->
-          <param name="initial_value">${initial_positions['shoulder_pan_joint']}</param>
+          <param name="initial_value">${initial_positions['ur_shoulder_pan_joint']}</param>
         </state_interface>
         <state_interface name="velocity"/>
@@ -91,5 +91,5 @@
         <state_interface name="position">
           <!-- initial position for the FakeSystem and simulation -->
-          <param name="initial_value">${initial_positions['shoulder_lift_joint']}</param>
+          <param name="initial_value">${initial_positions['ur_shoulder_lift_joint']}</param>
         </state_interface>
         <state_interface name="velocity"/>
@@ -107,5 +107,5 @@
         <state_interface name="position">
           <!-- initial position for the FakeSystem and simulation -->
-          <param name="initial_value">${initial_positions['elbow_joint']}</param>
+          <param name="initial_value">${initial_positions['ur_elbow_joint']}</param>
         </state_interface>
         <state_interface name="velocity"/>
@@ -123,5 +123,5 @@
         <state_interface name="position">
           <!-- initial position for the FakeSystem and simulation -->
-          <param name="initial_value">${initial_positions['wrist_1_joint']}</param>
+          <param name="initial_value">${initial_positions['ur_wrist_1_joint']}</param>
         </state_interface>
         <state_interface name="velocity"/>
@@ -139,5 +139,5 @@
         <state_interface name="position">
           <!-- initial position for the FakeSystem and simulation -->
-          <param name="initial_value">${initial_positions['wrist_2_joint']}</param>
+          <param name="initial_value">${initial_positions['ur_wrist_2_joint']}</param>
         </state_interface>
         <state_interface name="velocity"/>
@@ -155,5 +155,5 @@
         <state_interface name="position">
           <!-- initial position for the FakeSystem and simulation -->
-          <param name="initial_value">${initial_positions['wrist_3_joint']}</param>
+          <param name="initial_value">${initial_positions['ur_wrist_3_joint']}</param>
         </state_interface>
         <state_interface name="velocity"/>

File: Universal_Robots_ROS2_Description/urdf/ur_macro.xacro (robot description, xacro)
@@ -63,5 +63,5 @@
     sim_ignition:=false
     headless_mode:=false
-    initial_positions:=${dict(shoulder_pan_joint=0.0,shoulder_lift_joint=-1.57,elbow_joint=0.0,wrist_1_joint=-1.57,wrist_2_joint=0.0,wrist_3_joint=0.0)}
+    initial_positions:=${dict(ur_shoulder_pan_joint=0.0,ur_shoulder_lift_joint=-1.57,ur_elbow_joint=0.0,ur_wrist_1_joint=-1.57,ur_wrist_2_joint=0.0,ur_wrist_3_joint=0.0)}
     use_tool_communication:=false
     tool_voltage:=0
